File: MiSTer_A8SIO/MiSTer_A8SIO.kicad_sch (KiCad schematic)
At the start: 16 parts, among them J1 USB3_A, J2 SIO CONNECTOR, J3 Conn_01x10_Socket, J4 Conn_01x10_Socket, J5 Conn_01x02_Socket, J6 Conn_01x02_Socket, Q1 BC857, U1 TXS0108EPW, U2 AMS1117-3.3

Commit message: Ver. 1.2, Fixed crossed lines
Signed-off-by: Pawel Mandes <pawel.mandes@gmail>
Parts:
- removed C3, C4: 100nF, symbol Device:C_Small
- removed J3, J4: Conn_01x10_Socket, Connector_PinHeader_2.54mm:PinHeader_1x10_P2.54mm_Vertical, symbol Connector:Conn_01x10_Socket
- removed U1: TXS0108EPW, Package_SO:TSSOP-20_4.4x6.5mm_P0.65mm, symbol Logic_LevelTranslator:TXS0108EPW
- added J3, J4, J5, J6: Conn_01x06_Socket, Connector_PinHeader_2.54mm:PinHeader_1x06_P2.54mm_Vertical, symbol Connector:Conn_01x06_Socket
- J1: footprint Connector_USB:USB3_A_Molex_48393-001 -> Atari:USB3_A
- J7: renamed from J5; footprint Connector_PinSocket_2.54mm:PinSocket_1x02_P2.54mm_Vertical -> Connector_PinHeader_2.54mm:PinHeader_1x02_P2.54mm_Vertical
- J8: renamed from J6; footprint Connector_PinSocket_2.54mm:PinSocket_1x02_P2.54mm_Vertical -> Connector_PinHeader_2.54mm:PinHeader_1x02_P2.54mm_Vertical
- R1, R2: footprint Resistor_SMD:R_0603_1608Metric_Pad0.98x0.95mm_HandSolder -> Resistor_SMD:R_0805_2012Metric_Pad1.20x1.40mm_HandSolder
- U1: renamed from U2; footprint Package_TO_SOT_SMD:TO-252-3_TabPin2 -> Package_TO_SOT_SMD:SOT-223
Connections:
- net +3.3V: now also U1.4 (VO), J3.3 (Pin_3), J5.3 (Pin_3)
- net CLOCK IN: now also J4.6 (Pin_6)
- net COMMAND: now also J6.1 (Pin_1)
- net DATA IN: now also J6.5 (Pin_5)
- net DATA OUT: now also J6.2 (Pin_2)
- net GND: now also J3.4 (Pin_4), J4.4 (Pin_4), J5.4 (Pin_4), J6.4 (Pin_4)
- net INTERRUPT: now also J4.1 (Pin_1)
- net PRE_MOTOR: now also J4.5 (Pin_5)
- net PROCEED: now also J4.2 (Pin_2)
- net SIO_CLKIN_A: now also J3.6 (Pin_6)
- net SIO_CMD_A: now also J1.5 (SSRX-), J5.1 (Pin_1); no longer J1.8 (SSTX-)
- net SIO_IN_A: now also J5.5 (Pin_5)
- net SIO_IRQ_A: now also J1.8 (SSTX-), J3.1 (Pin_1); no longer J1.5 (SSRX-)
- net SIO_MOTOR_A: now also J1.6 (SSRX+), J3.5 (Pin_5); no longer J1.9 (SSTX+)
- net SIO_OUT_A: now also J5.2 (Pin_2)
- net SIO_PROC_A: now also J1.9 (SSTX+), J3.2 (Pin_2); no longer J1.6 (SSRX+)
- net VBUS: now also J4.3 (Pin_3), J6.3 (Pin_3)
- no-connect marks 7 -> 5
Other:
- note added: "HV1 HV2 HV GND HV3 HV4"
- note added: "LV1 LV2 LV GND LV3 LV4"
- note added: "MrFPGA P7 | USB Name | |Signal ----------+----------+---+------------- 0 | D+ | I |SIO_IN 1 | D- | O |SIO_OUT 4 | TX- | O |SIO_CMD 5 | GND_DRN | I |SIO_CLKIN 6 | RX+ | I |SIO_PROC 7 | RX- | I |SIO_IRQ 9 | TX+ | O |SIO_MOTOR USB3 A-A Cable crossed pairs: RX- (5) <----> TX- (8) RX+ (6) <----> TX+ (9) TX- (8) <----> RX- (5) TX+ (9) <----> TX- (6)"
- note removed: "Pin | USB Name | |Signal ----+----------+---+------------- 0 | D+ | I |SIO_IN 1 | D- | O |SIO_OUT 2 | TX- | O |SIO_CMD 3 | GND_d | I |SIO_CLKIN 4 | RX+ | I |SIO_PROC 5 | RX- | I |SIO_IRQ 6 | TX+ | O |SIO_MOTOR"
- moved on the sheet: J7, J8
